Commit message: full test completed : OK. TODO : add multiple other shapes...

File: models/GazeboDomainRandom/urdf/box.urdf.xacro (robot description, xacro)
@@ -5,21 +5,21 @@
 	<xacro:arg name="name" default="BOX1"/>
 	-->
-	<xacro:macro name="simple_box" params="name color">
+	<xacro:macro name="simple_box" params="name color scale">
 		<link name="box_${name}">
 		  <inertial>
-		    <origin xyz="2 0 0" />
+		    <origin xyz="0 0 0" />
 		    <mass value="10.0" />
 		    <inertia  ixx="1.0" ixy="0.0"  ixz="0.0"  iyy="100.0"  iyz="0.0"  izz="1.0" />
 		  </inertial>
 		  <visual>
-		    <origin xyz="2 0 1"/>
+		    <origin xyz="${scale*0.5} ${scale*0.5} ${scale*0.5}"/>
 		    <geometry>
-		      <box size="1 1 2" />
+		      <box size="${scale*1} ${scale*1} ${scale*1}" />
 		    </geometry>
 		  </visual>
 		  <collision>
-		    <origin xyz="2 0 1"/>
+		    <origin xyz="${scale*0.5} ${scale*0.5} ${scale*0.5}"/>
 		    <geometry>
-		      <box size="1 1 2" />
+		      <box size="${scale*1} ${scale*1} ${scale*1}" />
 		    </geometry>
 		  </collision>
@@ -29,4 +29,4 @@
 		</gazebo>
 	</xacro:macro>
-	<xacro:simple_box name="$(arg name)" color="$(arg color)"/>
+	<xacro:simple_box name="$(arg name)" color="$(arg color)" scale="$(arg scale)"/>
 </robot>
