Commit message: add a point light source... TODO : TEST further...

File: models/GazeboDomainRandom/urdf/cylinder.urdf.xacro (robot description, xacro)
@@ -13,13 +13,13 @@
 		  </inertial>
 		  <visual>
-		    <origin xyz="0 0 ${scale*0.25}"/>
+		    <origin xyz="0 0 ${scale*0.125}"/>
 		    <geometry>
-		      <cylinder radius="${scale*0.5}" length="${scale*0.5}" />
+		      <cylinder radius="${scale*0.25}" length="${scale*0.25}" />
 		    </geometry>
 		  </visual>
 		  <collision>
-		    <origin xyz="0 0 ${scale*0.25}"/>
+		    <origin xyz="0 0 ${scale*0.125}"/>
 		    <geometry>
-		      <cylinder radius="${scale*0.5}" length="${scale*0.5}" />
+		      <cylinder radius="${scale*0.25}" length="${scale*0.25}" />
 		    </geometry>
 		  </collision>

File: models/GazeboDomainRandom/urdf/rectangle.urdf.xacro (robot description, xacro)
@@ -13,13 +13,13 @@
 		  </inertial>
 		  <visual>
-		    <origin xyz="0 0 ${scale*0.25}"/>
+		    <origin xyz="0 0 ${scale*0.125}"/>
 		    <geometry>
-		      <box size="${scale*0.5} ${scale*1} ${scale*0.5}" />
+		      <box size="${scale*0.25} ${scale*0.5} ${scale*0.25}" />
 		    </geometry>
 		  </visual>
 		  <collision>
-		    <origin xyz="0 0 ${scale*0.25}"/>
+		    <origin xyz="0 0 ${scale*0.125}"/>
 		    <geometry>
-		      <box size="${scale*0.5} ${scale*1} ${scale*0.5}" />
+		      <box size="${scale*0.25} ${scale*0.5} ${scale*0.25}" />
 		    </geometry>
 		  </collision>

File: models/GazeboDomainRandom/urdf/sphere.urdf.xacro (robot description, xacro)
@@ -9,13 +9,13 @@
 		  </inertial>
 		  <visual>
-		    <origin xyz="0 0 ${scale*0.5}"/>
+		    <origin xyz="0 0 ${scale*0.25}"/>
 		    <geometry>
-		      <sphere radius="${scale*0.5}" />
+		      <sphere radius="${scale*0.25}" />
 		    </geometry>
 		  </visual>
 		  <collision>
-		    <origin xyz="0 0 ${scale*0.5}"/>
+		    <origin xyz="0 0 ${scale*0.25}"/>
 		    <geometry>
-		      <sphere radius="${scale*0.5}" />
+		      <sphere radius="${scale*0.25}" />
 		    </geometry>
 		  </collision>
